File: Z23.kicad_pcb (KiCad board)
At the start: 2 copper layers, 50 x 70 mm, 0 parts

Commit message: Added default sizes for traces and vias
Other:
- net class Default: clearance 0.2 -> 0.25; via_dia 0.8 -> 2; via_drill 0.4 -> 0.8
- rule trace_clearance: 0.2 -> 0.25
- rule trace_min: 0.2 -> 0.25
- rule via_min_drill: 0.3 -> 0.8
- rule via_min_size: 0.4 -> 2
Changed lines of the file:
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@@
   )
   (setup
-    (last_trace_width 0.25)
-    (trace_clearance 0.2)
+    (last_trace_width 0.5)
+    (user_trace_width 0.5)
+    (user_trace_width 0.75)
+    (user_trace_width 1)
+    (user_trace_width 1.5)
+    (user_trace_width 2)
+    (trace_clearance 0.25)
     (zone_clearance 0.508)
     (zone_45_only no)
-    (trace_min 0.2)
+    (trace_min 0.25)
     (segment_width 0.2)
     (edge_width 0.15)
-    (via_size 0.8)
-    (via_drill 0.4)
-    (via_min_size 0.4)
-    (via_min_drill 0.3)
+    (via_size 2)
+    (via_drill 0.8)
+    (via_min_size 2)
+    (via_min_drill 0.8)
     (uvia_size 0.3)
     (uvia_drill 0.1)
@@
     (mod_text_size 1 1)
     (mod_text_width 0.15)
-    (pad_size 1.524 1.524)
-    (pad_drill 0.762)
+    (pad_size 2.5 1.7)
+    (pad_drill 1)
     (pad_to_mask_clearance 0.051)
     (solder_mask_min_width 0.25)
@@
   (net 0 "")
   (net_class Default "This is the default net class."
-    (clearance 0.2)
+    (clearance 0.25)
     (trace_width 0.25)
-    (via_dia 0.8)
-    (via_drill 0.4)
+    (via_dia 2)
+    (via_drill 0.8)
     (uvia_dia 0.3)
     (uvia_drill 0.1)
+    (diff_pair_gap 0.25)
+    (diff_pair_width 0.25)
   )
   (target plus (at 50 108.5) (size 5) (width 0.15) (layer Edge.Cuts))
